Commit message: update xyz = [-0.05951 0.09345 0.09596] and rpy = [0.9 1 180.45]

File: syn_ur10_bringup/urdf/tool_b.urdf.xacro (robot description, xacro)
@@ -142,9 +142,9 @@
     <parent link="tool_base"/>
     <child link="camera_plate"/>
-    <origin xyz="-0.0392 0.0298 0.069" rpy="0 0 0" />
+    <origin xyz="-0.0392 0.0298 0.079" rpy="0 0 0" />
   </joint>
   <!-- scanCONTROL_2900-50 sensor and is connected to tool_base frame -->
   <xacro:scanCONTROL_2900-50 prefix="scanCONTROL_2900-50_" parent="tool_base">
-    <origin xyz="-0.060 0.09 0.078" rpy="${radians(0)} ${radians(0)} ${radians(180)}" />
+    <origin xyz="-0.05951 0.09345 0.09596" rpy="${radians(0.9)} ${radians(1)} ${radians(180.45)}" />
   </xacro:scanCONTROL_2900-50>
   <!-- camera_support link is connected to scanCONTROL_2900-50_scanner_link -->

Commit message: update tool position with [h, v] = [0.00485, 0.01575]

File: syn_ur10_bringup/urdf/tool_b.urdf.xacro (robot description, xacro)
@@ -2,9 +2,12 @@
 <robot xmlns:xacro="http://www.ros.org/wiki/xacro" name="tool">
   <!-- change the value of rivet_tool_distance_offset to adjust the distance to the target-->
-  <xacro:property name="rivet_tool_distance_offset" value="-0.0020" />
+  <!-- old value = -0.0020 -->
+  <xacro:property name="rivet_tool_distance_offset" value="0.0000" />
   <!-- change the value of rivet_tool_horizontal_adjust to adjust the tool horizontally, plus for left and minus for right -->
-  <xacro:property name="rivet_tool_horizontal_adjust" value="0.0017" />
+  <!-- old value = 0.00485 -->
+  <xacro:property name="rivet_tool_horizontal_adjust" value="0.00485" />
   <!-- change the value of rivet_tool_vertical_adjust to adjust the tool vertically, plus for up and minus for down -->
-  <xacro:property name="rivet_tool_vertical_adjust" value="0.0004" />
+  <!-- old value = 0.01575 -->
+  <xacro:property name="rivet_tool_vertical_adjust" value="0.01575" />
   <xacro:include filename="$(find microepsilon_scancontrol)/description/urdf/scanCONTROL_2900-50_macro.urdf.xacro" />
   <xacro:property name="rivet_tool_part_1_length" value="0.05078" />

Commit message: update [rivet_tool_horizontal_adjust] to [0.0044]

File: syn_ur10_bringup/urdf/tool_b.urdf.xacro (robot description, xacro)
@@ -6,8 +6,8 @@
   <!-- change the value of rivet_tool_horizontal_adjust to adjust the tool horizontally, plus for left and minus for right -->
   <!-- old value = 0.00485 -->
-  <xacro:property name="rivet_tool_horizontal_adjust" value="0.00485" />
+  <xacro:property name="rivet_tool_horizontal_adjust" value="0.0044" />
   <!-- change the value of rivet_tool_vertical_adjust to adjust the tool vertically, plus for up and minus for down -->
   <!-- old value = 0.01575 -->
-  <xacro:property name="rivet_tool_vertical_adjust" value="0.01575" />
+  <xacro:property name="rivet_tool_vertical_adjust" value="0.0165" />
   <xacro:include filename="$(find microepsilon_scancontrol)/description/urdf/scanCONTROL_2900-50_macro.urdf.xacro" />
   <xacro:property name="rivet_tool_part_1_length" value="0.05078" />
