Commit message: fix the orientation of [tool_base], set [yaw] to [180]

File: syn_ur10_bringup/urdf/syn_ur10_setup.urdf.xacro (robot description, xacro)
@@ -28,5 +28,5 @@
     <parent link="ur10_tool0" />
     <child link = "tool_base" />
-    <origin xyz="0.0 0.0 0.0" rpy="0.0 0.0 0.0" />
+    <origin xyz="0.0 0.0 0.0" rpy="0.0 0.0 ${radians(180)}" />
   </joint>
 </robot>
