Commit message: change the rivet_tool_horizontal_adjust and rivet_tool_vertical_adjust parameters

File: syn_ur10_bringup/urdf/tool.urdf.xacro (robot description, xacro)
@@ -2,9 +2,9 @@
 <robot xmlns:xacro="http://www.ros.org/wiki/xacro" name="tool">
   <!-- change the value of rivet_tool_distance_offset to adjust the distance to the target-->
-  <xacro:property name="rivet_tool_distance_offset" value="0.0000" />
+  <xacro:property name="rivet_tool_distance_offset" value="-0.0020" />
   <!-- change the value of rivet_tool_horizontal_adjust to adjust the tool horizontally, plus for left and minus for right -->
-  <xacro:property name="rivet_tool_horizontal_adjust" value="-0.0047" />
+  <xacro:property name="rivet_tool_horizontal_adjust" value="0.0058" />
   <!-- change the value of rivet_tool_vertical_adjust to adjust the tool vertically, plus for up and minus for down -->
-  <xacro:property name="rivet_tool_vertical_adjust" value="-0.0015" />
+  <xacro:property name="rivet_tool_vertical_adjust" value="0.0030" />
   <xacro:include filename="$(find microepsilon_scancontrol)/description/urdf/scanCONTROL_2900-50_macro.urdf.xacro" />
   <xacro:property name="rivet_tool_part_1_length" value="0.05078" />
@@ -60,5 +60,5 @@
     <child link="rivet_tool_part_1"/>
     <!-- <origin xyz="0 -0.03275 ${0.03787 + rivet_tool_z_adjust}" rpy="${radians(90)} 0 0" /> -->
-    <origin xyz="${0 - rivet_tool_horizontal_adjust} -0.03275 ${0.03787 - rivet_tool_vertical_adjust}" rpy="${radians(90)} ${radians(rivet_tool_angle)} 0" />
+    <origin xyz="${0 + rivet_tool_horizontal_adjust} -0.03275 ${0.03787 + rivet_tool_vertical_adjust}" rpy="${radians(90)} ${radians(rivet_tool_angle)} 0" />
   </joint>
   <link name="rivet_tool_part_2">

Commit message: adjust the position of the rivet tool

File: syn_ur10_bringup/urdf/tool.urdf.xacro (robot description, xacro)
@@ -4,7 +4,7 @@
   <xacro:property name="rivet_tool_distance_offset" value="-0.0020" />
   <!-- change the value of rivet_tool_horizontal_adjust to adjust the tool horizontally, plus for left and minus for right -->
-  <xacro:property name="rivet_tool_horizontal_adjust" value="0.0058" />
+  <xacro:property name="rivet_tool_horizontal_adjust" value="0.0008" />
   <!-- change the value of rivet_tool_vertical_adjust to adjust the tool vertically, plus for up and minus for down -->
-  <xacro:property name="rivet_tool_vertical_adjust" value="0.0030" />
+  <xacro:property name="rivet_tool_vertical_adjust" value="0.0004" />
   <xacro:include filename="$(find microepsilon_scancontrol)/description/urdf/scanCONTROL_2900-50_macro.urdf.xacro" />
   <xacro:property name="rivet_tool_part_1_length" value="0.05078" />

Commit message: update the rivet tool position parameters

File: syn_ur10_bringup/urdf/tool.urdf.xacro (robot description, xacro)
@@ -4,7 +4,7 @@
   <xacro:property name="rivet_tool_distance_offset" value="-0.0020" />
   <!-- change the value of rivet_tool_horizontal_adjust to adjust the tool horizontally, plus for left and minus for right -->
-  <xacro:property name="rivet_tool_horizontal_adjust" value="0.0008" />
+  <xacro:property name="rivet_tool_horizontal_adjust" value="0.0058" />
   <!-- change the value of rivet_tool_vertical_adjust to adjust the tool vertically, plus for up and minus for down -->
-  <xacro:property name="rivet_tool_vertical_adjust" value="0.0004" />
+  <xacro:property name="rivet_tool_vertical_adjust" value="0.00249" />
   <xacro:include filename="$(find microepsilon_scancontrol)/description/urdf/scanCONTROL_2900-50_macro.urdf.xacro" />
   <xacro:property name="rivet_tool_part_1_length" value="0.05078" />

Commit message: new [rivet_tool_vertical_adjust] = 0.0024

File: syn_ur10_bringup/urdf/tool.urdf.xacro (robot description, xacro)
@@ -6,5 +6,5 @@
   <xacro:property name="rivet_tool_horizontal_adjust" value="0.0058" />
   <!-- change the value of rivet_tool_vertical_adjust to adjust the tool vertically, plus for up and minus for down -->
-  <xacro:property name="rivet_tool_vertical_adjust" value="0.00249" />
+  <xacro:property name="rivet_tool_vertical_adjust" value="0.00240" />
   <xacro:include filename="$(find microepsilon_scancontrol)/description/urdf/scanCONTROL_2900-50_macro.urdf.xacro" />
   <xacro:property name="rivet_tool_part_1_length" value="0.05078" />

Commit message: update the pose of the laser scanner and update the [H, V] to [0.0058, 0.0155]

File: syn_ur10_bringup/urdf/tool.urdf.xacro (robot description, xacro)
@@ -2,9 +2,12 @@
 <robot xmlns:xacro="http://www.ros.org/wiki/xacro" name="tool">
   <!-- change the value of rivet_tool_distance_offset to adjust the distance to the target-->
-  <xacro:property name="rivet_tool_distance_offset" value="-0.0020" />
+  <!-- old value = -0.0020 -->
+  <xacro:property name="rivet_tool_distance_offset" value="0.0000" />
   <!-- change the value of rivet_tool_horizontal_adjust to adjust the tool horizontally, plus for left and minus for right -->
-  <xacro:property name="rivet_tool_horizontal_adjust" value="0.0058" />
+  <!-- old value = 0.00485 -->
+  <xacro:property name="rivet_tool_horizontal_adjust" value="0.0046" />
   <!-- change the value of rivet_tool_vertical_adjust to adjust the tool vertically, plus for up and minus for down -->
-  <xacro:property name="rivet_tool_vertical_adjust" value="0.00240" />
+  <!-- old value = 0.01575 -->
+  <xacro:property name="rivet_tool_vertical_adjust" value="0.0155" />
   <xacro:include filename="$(find microepsilon_scancontrol)/description/urdf/scanCONTROL_2900-50_macro.urdf.xacro" />
   <xacro:property name="rivet_tool_part_1_length" value="0.05078" />
@@ -142,9 +145,9 @@
     <parent link="tool_base"/>
     <child link="camera_plate"/>
-    <origin xyz="-0.0392 0.0298 0.069" rpy="0 0 0" />
+    <origin xyz="-0.0392 0.0298 0.079" rpy="0 0 0" />
   </joint>
   <!-- scanCONTROL_2900-50 sensor and is connected to tool_base frame -->
   <xacro:scanCONTROL_2900-50 prefix="scanCONTROL_2900-50_" parent="tool_base">
-    <origin xyz="-0.060 0.09 0.078" rpy="${radians(0)} ${radians(0)} ${radians(180)}" />
+    <origin xyz="-0.05951 0.09345 0.09596" rpy="${radians(0.9)} ${radians(1)} ${radians(180.45)}" />
   </xacro:scanCONTROL_2900-50>
   <!-- camera_support link is connected to scanCONTROL_2900-50_scanner_link -->

Commit message: update [h, v] to [0.0050, 0.0152]

File: syn_ur10_bringup/urdf/tool.urdf.xacro (robot description, xacro)
@@ -3,11 +3,11 @@
   <!-- change the value of rivet_tool_distance_offset to adjust the distance to the target-->
   <!-- old value = -0.0020 -->
-  <xacro:property name="rivet_tool_distance_offset" value="0.0000" />
+  <xacro:property name="rivet_tool_distance_offset" value="0.0013" />
   <!-- change the value of rivet_tool_horizontal_adjust to adjust the tool horizontally, plus for left and minus for right -->
-  <!-- old value = 0.00485 -->
-  <xacro:property name="rivet_tool_horizontal_adjust" value="0.0046" />
+  <!-- old value = 0.0046 -->
+  <xacro:property name="rivet_tool_horizontal_adjust" value="0.0050" />
   <!-- change the value of rivet_tool_vertical_adjust to adjust the tool vertically, plus for up and minus for down -->
-  <!-- old value = 0.01575 -->
-  <xacro:property name="rivet_tool_vertical_adjust" value="0.0155" />
+  <!-- old value = 0.0155 -->
+  <xacro:property name="rivet_tool_vertical_adjust" value="0.0152" />
   <xacro:include filename="$(find microepsilon_scancontrol)/description/urdf/scanCONTROL_2900-50_macro.urdf.xacro" />
   <xacro:property name="rivet_tool_part_1_length" value="0.05078" />

Commit message: set [rivet_tool_vertical_adjust] to [0.0150]

File: syn_ur10_bringup/urdf/tool.urdf.xacro (robot description, xacro)
@@ -8,6 +8,6 @@
   <xacro:property name="rivet_tool_horizontal_adjust" value="0.0050" />
   <!-- change the value of rivet_tool_vertical_adjust to adjust the tool vertically, plus for up and minus for down -->
-  <!-- old value = 0.0155 -->
-  <xacro:property name="rivet_tool_vertical_adjust" value="0.0152" />
+  <!-- old value = 0.0155 0.0152 -->
+  <xacro:property name="rivet_tool_vertical_adjust" value="0.0150" />
   <xacro:include filename="$(find microepsilon_scancontrol)/description/urdf/scanCONTROL_2900-50_macro.urdf.xacro" />
   <xacro:property name="rivet_tool_part_1_length" value="0.05078" />

Commit message: restore [v] to [0.0152]

File: syn_ur10_bringup/urdf/tool.urdf.xacro (robot description, xacro)
@@ -8,6 +8,6 @@
   <xacro:property name="rivet_tool_horizontal_adjust" value="0.0050" />
   <!-- change the value of rivet_tool_vertical_adjust to adjust the tool vertically, plus for up and minus for down -->
-  <!-- old value = 0.0155 0.0152 -->
-  <xacro:property name="rivet_tool_vertical_adjust" value="0.0150" />
+  <!-- old value = 0.0155 -->
+  <xacro:property name="rivet_tool_vertical_adjust" value="0.0152" />
   <xacro:include filename="$(find microepsilon_scancontrol)/description/urdf/scanCONTROL_2900-50_macro.urdf.xacro" />
   <xacro:property name="rivet_tool_part_1_length" value="0.05078" />

Commit message: set [h, v] to [0.0047, 0.0160]

File: syn_ur10_bringup/urdf/tool.urdf.xacro (robot description, xacro)
@@ -5,9 +5,9 @@
   <xacro:property name="rivet_tool_distance_offset" value="0.0013" />
   <!-- change the value of rivet_tool_horizontal_adjust to adjust the tool horizontally, plus for left and minus for right -->
-  <!-- old value = 0.0046 -->
-  <xacro:property name="rivet_tool_horizontal_adjust" value="0.0050" />
+  <!-- old value = 0.0046 0.0050 -->
+  <xacro:property name="rivet_tool_horizontal_adjust" value="0.0047" />
   <!-- change the value of rivet_tool_vertical_adjust to adjust the tool vertically, plus for up and minus for down -->
-  <!-- old value = 0.0155 -->
-  <xacro:property name="rivet_tool_vertical_adjust" value="0.0152" />
+  <!-- old value = 0.0155 0.0152 -->
+  <xacro:property name="rivet_tool_vertical_adjust" value="0.0160" />
   <xacro:include filename="$(find microepsilon_scancontrol)/description/urdf/scanCONTROL_2900-50_macro.urdf.xacro" />
   <xacro:property name="rivet_tool_part_1_length" value="0.05078" />

Commit message: use the new end-effector model

File: syn_ur10_bringup/urdf/tool.urdf.xacro (robot description, xacro)
@@ -3,20 +3,20 @@
   <!-- change the value of rivet_tool_distance_offset to adjust the distance to the target-->
   <!-- old value = -0.0020 -->
-  <xacro:property name="rivet_tool_distance_offset" value="0.0013" />
+  <xacro:property name="rivet_tool_distance_offset" value="0.00" />
   <!-- change the value of rivet_tool_horizontal_adjust to adjust the tool horizontally, plus for left and minus for right -->
   <!-- old value = 0.0046 0.0050 -->
-  <xacro:property name="rivet_tool_horizontal_adjust" value="0.0047" />
+  <xacro:property name="rivet_tool_horizontal_adjust" value="-0.013" />
   <!-- change the value of rivet_tool_vertical_adjust to adjust the tool vertically, plus for up and minus for down -->
   <!-- old value = 0.0155 0.0152 -->
-  <xacro:property name="rivet_tool_vertical_adjust" value="0.0160" />
+  <xacro:property name="rivet_tool_vertical_adjust" value="-0.007" />
   <xacro:include filename="$(find microepsilon_scancontrol)/description/urdf/scanCONTROL_2900-50_macro.urdf.xacro" />
   <xacro:property name="rivet_tool_part_1_length" value="0.05078" />
   <xacro:property name="rivet_tool_part_1_radius" value="0.015" />
   <xacro:property name="rivet_tool_part_2_height" value="0.012" />
-  <xacro:property name="rivet_tool_part_2_length" value="0.066" />
+  <xacro:property name="rivet_tool_part_2_length" value="0.088" />
   <xacro:property name="rivet_tool_part_2_width" value="0.03" />
   <xacro:property name="rivet_tool_part_3_length" value="0.06374" />
   <xacro:property name="rivet_tool_part_3_radius" value="0.0075" />
-  <xacro:property name="rivet_tool_angle" value="154.6" />
+  <xacro:property name="rivet_tool_angle" value="155.2" />
   <link name="tool_base">
     <inertial>
@@ -27,13 +27,13 @@
     <visual>
       <material name="lightgray" />
-      <origin xyz="0.0 0.0 0.03725" />
+      <origin xyz="0.0 0.0 0.0604" />
       <geometry>
-        <box size="0.070 0.0655 0.0705" />
+        <box size="0.070 0.0655 0.1208" />
       </geometry>
     </visual>
     <collision>
-      <origin xyz="0.0 0.0 0.03725" />
+      <origin xyz="0.0 0.0 0.0604" />
       <geometry>
-        <box size="0.070 0.0655 0.0705" />
+        <box size="0.070 0.0655 0.1208" />
       </geometry>
     </collision>
@@ -59,9 +59,15 @@
     </collision>
   </link>
+  <link name="rivet_base" />
+  <joint name="tool_base_rivet_base_joint" type="fixed">
+    <parent link="tool_base"/>
+    <child link="rivet_base"/>
+    <origin xyz="0 -0.03275 0.09423" rpy="${radians(180)} 0 0"/>
+  </joint>
   <joint name="tool_base_rivet_tool_part_1_joint" type="fixed">
     <parent link="tool_base"/>
     <child link="rivet_tool_part_1"/>
     <!-- <origin xyz="0 -0.03275 ${0.03787 + rivet_tool_z_adjust}" rpy="${radians(90)} 0 0" /> -->
-    <origin xyz="${0 + rivet_tool_horizontal_adjust} -0.03275 ${0.03787 + rivet_tool_vertical_adjust}" rpy="${radians(90)} ${radians(rivet_tool_angle)} 0" />
+    <origin xyz="${0 + rivet_tool_horizontal_adjust} -0.03275 ${0.09423 + rivet_tool_vertical_adjust}" rpy="${radians(90)} ${radians(rivet_tool_angle)} 0"/>
   </joint>
   <link name="rivet_tool_part_2">
@@ -132,5 +138,5 @@
       <origin xyz="0.0 0.0 0.0" />
       <geometry>
-        <box size="0.003 0.126 0.132" />
+        <box size="0.003 0.126 0.162" />
       </geometry>
     </visual>
@@ -138,5 +144,5 @@
       <origin xyz="0.0 0.0 0.0" />
       <geometry>
-        <box size="0.003 0.126 0.132" />
+        <box size="0.003 0.126 0.162" />
       </geometry>
     </collision>
@@ -145,9 +151,9 @@
     <parent link="tool_base"/>
     <child link="camera_plate"/>
-    <origin xyz="-0.0392 0.0298 0.079" rpy="0 0 0" />
+    <origin xyz="-0.0382 0.0298 0.079" rpy="0 0 0" />
   </joint>
   <!-- scanCONTROL_2900-50 sensor and is connected to tool_base frame -->
   <xacro:scanCONTROL_2900-50 prefix="scanCONTROL_2900-50_" parent="tool_base">
-    <origin xyz="-0.05951 0.09345 0.09596" rpy="${radians(0.9)} ${radians(1)} ${radians(180.45)}" />
+    <origin xyz="-0.05755 0.08971 0.10693" rpy="${radians(1.3)} ${radians(0)} ${radians(180)}" />
   </xacro:scanCONTROL_2900-50>
   <!-- camera_support link is connected to scanCONTROL_2900-50_scanner_link -->

Commit message: change [h] to [-0.015]

File: syn_ur10_bringup/urdf/tool.urdf.xacro (robot description, xacro)
@@ -6,5 +6,5 @@
   <!-- change the value of rivet_tool_horizontal_adjust to adjust the tool horizontally, plus for left and minus for right -->
   <!-- old value = 0.0046 0.0050 -->
-  <xacro:property name="rivet_tool_horizontal_adjust" value="-0.013" />
+  <xacro:property name="rivet_tool_horizontal_adjust" value="-0.015" />
   <!-- change the value of rivet_tool_vertical_adjust to adjust the tool vertically, plus for up and minus for down -->
   <!-- old value = 0.0155 0.0152 -->

Commit message: find realsense model from package [realsense2_description] instead of [realsense2_camera]

File: syn_ur10_bringup/urdf/tool.urdf.xacro (robot description, xacro)
@@ -1,4 +1,4 @@
 <?xml version="1.0"?>
-<robot xmlns:xacro="http://www.ros.org/wiki/xacro" name="tool">
+<robot name="tool" xmlns:xacro="http://ros.org/wiki/xacro">
   <!-- change the value of rivet_tool_distance_offset to adjust the distance to the target-->
   <!-- old value = -0.0020 -->
@@ -190,7 +190,8 @@
   </joint>
   <!-- connect camera to link camera_support_2 -->
-  <xacro:include filename="$(find realsense2_camera)/urdf/_r430.urdf.xacro"/>
+  <xacro:include filename="$(find realsense2_description)/urdf/_r430.urdf.xacro" />
   <sensor_r430 parent="camera_support_2">
     <origin xyz="-0.0225 0 0" rpy="0 0 ${radians(90)}"/>
+    <!-- <origin xyz="0 0 0" rpy="0 0 ${radians(0)}"/> -->
   </sensor_r430>
 </robot>

Commit message: rename link [camera_support_2] to [rs_base_link] and fix the realsense D435 camera model problem (_r430.urdf.xacro to _d435.urdf.xacro)

File: syn_ur10_bringup/urdf/tool.urdf.xacro (robot description, xacro)
@@ -183,15 +183,13 @@
     <origin xyz="0 0.09 0.045" rpy="0.0 ${radians(90)} 0.0" />
   </joint>
-  <link name="camera_support_2" />
-  <joint name="camera_support_2_camera_support_joint" type="fixed">
+  <link name="rs_base_link" />
+  <joint name="rs_base_link_camera_support_joint" type="fixed">
     <parent link="camera_support"/>
-    <child link="camera_support_2"/>
+    <child link="rs_base_link"/>
     <origin xyz="0 0.0 0.0208" rpy="0.0 ${radians(0)} ${radians(180)}" />
   </joint>
-  <!-- connect camera to link camera_support_2 -->
-  <xacro:include filename="$(find realsense2_description)/urdf/_r430.urdf.xacro" />
-  <sensor_r430 parent="camera_support_2">
-    <origin xyz="-0.0225 0 0" rpy="0 0 ${radians(90)}"/>
-    <!-- <origin xyz="0 0 0" rpy="0 0 ${radians(0)}"/> -->
-  </sensor_r430>
+  <xacro:include filename="$(find realsense2_description)/urdf/_d435.urdf.xacro" />
+  <sensor_d435 parent="rs_base_link">
+    <origin xyz="0 0 0" rpy="0 0 ${radians(90)}"/>
+  </sensor_d435>
 </robot>

Commit message: set new [h, w] = [-0.0078 -0.0083]

File: syn_ur10_bringup/urdf/tool.urdf.xacro (robot description, xacro)
@@ -5,9 +5,9 @@
   <xacro:property name="rivet_tool_distance_offset" value="0.00" />
   <!-- change the value of rivet_tool_horizontal_adjust to adjust the tool horizontally, plus for left and minus for right -->
-  <!-- old value = 0.0046 0.0050 -->
-  <xacro:property name="rivet_tool_horizontal_adjust" value="-0.015" />
+  <!-- old value = -0.015 (15 degree)-->
+  <xacro:property name="rivet_tool_horizontal_adjust" value="-0.0078" />
   <!-- change the value of rivet_tool_vertical_adjust to adjust the tool vertically, plus for up and minus for down -->
-  <!-- old value = 0.0155 0.0152 -->
-  <xacro:property name="rivet_tool_vertical_adjust" value="-0.007" />
+  <!-- old value = -0.007 (15 degree)-->
+  <xacro:property name="rivet_tool_vertical_adjust" value="-0.0083" />
   <xacro:include filename="$(find microepsilon_scancontrol)/description/urdf/scanCONTROL_2900-50_macro.urdf.xacro" />
   <xacro:property name="rivet_tool_part_1_length" value="0.05078" />
