Commit message: update the urdf model for the robot

File: syn_ur10_bringup/urdf/syn_table.urdf.xacro (robot description, xacro)
@@ -3,11 +3,11 @@
   <xacro:arg name="floating_table" default="false" />
   <xacro:property name="roomheight" value="3.0" />
-  <xacro:property name="tableheight" value="0.83" />
-  <xacro:property name="tablewidth" value="0.83" />
-  <xacro:property name="tabledepth" value="0.9" />
-  <xacro:property name="ur10_mount_offset_y" value="-0.212" />
-  <xacro:property name="scan_offset_x" value="0.00" />
+  <xacro:property name="tableheight" value="0.855" />
+  <xacro:property name="tablewidth" value="0.60" />
+  <xacro:property name="tabledepth" value="0.905" />
+  <xacro:property name="ur10_mount_offset_y" value="-0.2585" />
+  <!-- <xacro:property name="scan_offset_x" value="0.00" />
   <xacro:property name="scan_offset_y" value="-0.40" />
-  <xacro:property name="scan_offset_z" value="0.06" />
+  <xacro:property name="scan_offset_z" value="0.06" /> -->
   <material name="white">
     <color rgba="1 1 1 1"/>
@@ -79,6 +79,25 @@
   </gazebo>
   <link name="table_top"/>
-  <link name="ur10_mount"/>
-  <link name="scan">
+  <link name="ur10_mount">
+    <visual>
+      <origin xyz="${0} ${0} ${0}" rpy="${0} ${0} ${0}"/>
+      <geometry>
+        <mesh filename="package://syn_ur10_bringup/meshes/ur10_mount.stl" scale="0.001 0.001 0.001"/>
+      </geometry>
+      <material name="aluminum"/>
+    </visual>
+    <collision>
+      <origin xyz="${0} ${0} ${0}" rpy="${0} ${0} ${0}"/>
+      <geometry>
+        <mesh filename="package://syn_ur10_bringup/meshes/ur10_mount.stl" scale="0.001 0.001 0.001"/>
+      </geometry>
+    </collision>
+    <inertial>
+      <mass value="0.300" />
+      <origin xyz="0 0 0.05" />
+      <inertia ixx="1.0" ixy="1.0" ixz="1.0" iyy="0.0" iyz="0.0" izz="0.0" />
+    </inertial>
+  </link>
+  <!-- <link name="scan">
     <inertial>
       <origin xyz="0.0 0.0 0.0" />
@@ -99,5 +118,5 @@
       </geometry>
     </collision>
-  </link>
+  </link> -->
   <joint name="table_floor_joint" type="floating">
     <parent link="floor"/>
@@ -115,8 +134,8 @@
 	  <origin xyz="0 ${ur10_mount_offset_y} 0" rpy="0 0 0" />
   </joint>
-  <joint name="scan_table_top_joint" type="fixed">
+  <!-- <joint name="scan_table_top_joint" type="fixed">
     <parent link="table_top"/>
     <child link="scan"/>
 	  <origin xyz="${scan_offset_x} ${scan_offset_y} ${scan_offset_z}" rpy="0 0 0" />
-  </joint>
+  </joint> -->
 </robot>

File: syn_ur10_bringup/urdf/syn_ur10_setup.urdf.xacro (robot description, xacro)
@@ -7,5 +7,5 @@
   <!-- tool -->
   <xacro:include filename="$(find syn_ur10_bringup)/urdf/tool.new.urdf.xacro" />
-  <xacro:property name="ur10_mount_height" value="0.01" />
+  <xacro:property name="ur10_mount_height" value="0.055" />
   <link name="world" />
   <joint name="floor_world_joint" type="fixed">
@@ -23,5 +23,5 @@
     <parent link="ur10_mount" />
     <child link = "ur10_base_link" />
-    <origin xyz="0.0 0.0 ${ur10_mount_height}" rpy="0.0 0.0 ${radians(90)}" />
+    <origin xyz="0.0 0.0 ${ur10_mount_height}" rpy="0.0 0.0 ${radians(-90)}" />
   </joint>
   <joint name="ur10_tool_joint" type="fixed">

File: syn_ur10_bringup/urdf/tool.new.urdf.xacro (robot description, xacro)
@@ -10,13 +10,13 @@
   <!-- old value = -0.007 (15 degree)-->
   <xacro:property name="rivet_tool_vertical_adjust" value="-0.0083" />
-  <xacro:property name="rivet_tool_x" value="0.00370" />
-  <xacro:property name="rivet_tool_y" value="0.21127" />
-  <xacro:property name="rivet_tool_z" value="0.17890" />
-  <xacro:property name="laser_x" value="-0.04399" />
-  <xacro:property name="laser_y" value="-0.12500" />
-  <xacro:property name="laser_z" value="0.14095" />
-  <xacro:property name="camera_x" value="0.01369" />
-  <xacro:property name="camera_y" value="0.06792" />
-  <xacro:property name="camera_z" value="0.01050" />
+  <xacro:property name="rivet_tool_x" value="0.00381" />
+  <xacro:property name="rivet_tool_y" value="0.217767" />
+  <xacro:property name="rivet_tool_z" value="0.1809" />
+  <xacro:property name="laser_x" value="-0.047604" />
+  <xacro:property name="laser_y" value="-0.118435" />
+  <xacro:property name="laser_z" value="0.147048" />
+  <xacro:property name="camera_x" value="0.013848" />
+  <xacro:property name="camera_y" value="0.07692" />
+  <xacro:property name="camera_z" value="0.0085" />
   <xacro:property name="camera_angle" value="90.00" />
   <link name="tool_base" />
@@ -25,5 +25,5 @@
       <origin xyz="${0} ${0} ${0}" rpy="${0} ${0} ${0}"/>
       <geometry>
-        <mesh filename="package://syn_ur10_bringup/meshes/Endeffektor.stl" scale="0.01 0.01 0.01"/>
+        <mesh filename="package://syn_ur10_bringup/meshes/Endeffektor.stl" scale="1 1 1"/>
       </geometry>
       <material name="aluminum"/>
@@ -32,5 +32,5 @@
       <origin xyz="${0} ${0} ${0}" rpy="${0} ${0} ${0}"/>
       <geometry>
-        <mesh filename="package://syn_ur10_bringup/meshes/Endeffektor.stl" scale="0.01 0.01 0.01"/>
+        <mesh filename="package://syn_ur10_bringup/meshes/Endeffektor.stl" scale="1 1 1"/>
       </geometry>
     </collision>

Commit message: change [table_floor_joint] to [fixed], remove the node [tf_dummy], and change [MoveGroupExecuteService] to [MoveGroupExecuteTrajectoryAction]

File: syn_ur10_bringup/urdf/syn_table.urdf.xacro (robot description, xacro)
@@ -119,5 +119,5 @@
     </collision>
   </link> -->
-  <joint name="table_floor_joint" type="floating">
+  <joint name="table_floor_joint" type="fixed">
     <parent link="floor"/>
     <child link="table"/>
